File: Striduino.kicad_pcb (KiCad board)
At the start: 2 copper layers, 100 x 36.5 mm, 45 parts, among them J1 SG90, J2 PERIP., J3 I2C, J4 SPI/STEPPER, J5 PWR, J7 Barrel_Jack, SW1 SW_SPST, SW2 Rotary_Encoder_Switch, U1 WC1602A, U2 AZ1117-5.0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

Commit message: Ordered PCB V1.0
Order boards to home for dec. ordered ali to ON for jan. wait till then to test around.
Parts:
- added Logo1: x, Symbol:ESD-Logo_6.6x6mm_SilkScreen, F.Cu at (60.5, 145.5)
- added Logo10: x, pics:chip, B.Cu at (132.2, 141.6)
- added Logo11: x, pics:bolt, B.Cu at (147.3, 120.1)
- added Logo2: x, Symbol:KiCad-Logo2_8mm_SilkScreen, F.Cu at (64.0, 126.8)
- added Logo3: x, pics:datboi, B.Cu at (112.8, 131.9)
- added Logo4: x, pics:stride, B.Cu at (71.4, 127.5)
- added Logo5: x, Symbol:ESD-Logo_6.6x6mm_SilkScreen, B.Cu at (101.2, 118.9)
- added Logo6: x, µ104KiCAD:SN_BLOCK, F.Cu at (81.6, 129.4)
- added Logo7: x, pics:datboi, F.Cu at (132.0, 145.9)
- added Logo8: x, µ104KiCAD:SN_BLOCK, B.Cu at (139.5, 133.8)
- added Logo9: x, pics:bolt, F.Cu at (127.5, 132.8)
Other:
- board text added: "(c) Mitchell Stride Striduino PN: 30-2019-002 v1.0 SN:"
- board text added: "|+V 5V 3V3 GND|"
- board text added: "|3V3 SDA SCL GND|"
- board text added: "|5V SCK MISO MOSI SS GND|"
- board text added: "|GND 5V A2|"
- board text added: "|GND A3 5V|"
- board text removed: "(c) Paradigm Hyperloop GeneralMCU PCB PN: 2019-001 v1.0 SN:"
